Commit message: Revert "squash commits together"
This reverts commit ba11b361a6fa3346667bb6310b62452d4b281266.

File: fanuc_lrmate200id_support/urdf/lrmate200id.xacro (robot description, xacro)
@@ -1,4 +1,4 @@
 <?xml version="1.0"?>
-<robot name="fanuc_lrmate200id" xmlns:xacro="http://wiki.ros.org/xacro">
+<robot name="fanuc_lrmate200id" xmlns:xacro="http://ros.org/wiki/xacro">
   <xacro:include filename="$(find fanuc_lrmate200id_support)/urdf/lrmate200id_macro.xacro"/>
   <xacro:fanuc_lrmate200id prefix=""/>

File: fanuc_lrmate200id_support/urdf/lrmate200id_macro.xacro (robot description, xacro)
@@ -1,7 +1,7 @@
 <?xml version="1.0"?>
-<robot xmlns:xacro="http://www.ros.org/wiki/xacro">
-  <xacro:include filename="$(find fanuc_lrmate200id_support)/urdf/common_materials.xacro"/>
+<robot xmlns:xacro="http://ros.org/wiki/xacro">
+  <xacro:include filename="$(find fanuc_resources)/urdf/common_materials.xacro"/>
+  <xacro:include filename="$(find fanuc_resources)/urdf/common_constants.xacro"/>
   <xacro:macro name="fanuc_lrmate200id" params="prefix">
-    <!-- links: main serial chain -->
     <link name="${prefix}base_link">
       <visual>
@@ -18,11 +18,4 @@
         </geometry>
       </collision>
-      <inertial>
-          <mass value="10.733459"/>
-          <origin xyz="0.014288 0.000001 0.122264" rpy="0.0 0.0 0.0"/>
-          <inertia ixx="0.096590" ixy="-0.000005" ixz="-0.003803"
-                                  iyy="0.087591"  iyz="-0.000001"
-                                                  izz="0.081632"/>
-      </inertial>
     </link>
     <link name="${prefix}link_1">
@@ -40,11 +33,4 @@
         </geometry>
       </collision>
-      <inertial>
-          <mass value="16.934564"/>
-          <origin xyz="0.019143 0.024764 -0.064596" rpy="0.0 0.0 0.0"/>
-          <inertia ixx="0.222318" ixy="0.016499" ixz="0.023794"
-                                  iyy="0.208959" iyz="0.031663"
-                                                 izz="0.157081"/>
-      </inertial>
     </link>
     <link name="${prefix}link_2">
@@ -62,11 +48,4 @@
         </geometry>
       </collision>
-      <inertial>
-          <mass value="12.98711"/>
-          <origin xyz="-0.000008 0.221181 0.173052" rpy="0.0 0.0 0.0"/>
-          <inertia ixx="0.425299" ixy="0.000005" ixz="-0.000004"
-                                  iyy="0.452311" iyz="-0.002920"
-                                                 izz="0.054493"/>
-      </inertial>
     </link>
     <link name="${prefix}link_3">
@@ -84,11 +63,4 @@
         </geometry>
       </collision>
-      <inertial>
-          <mass value="7.50151"/>
-          <origin xyz="0.000002 0.065008 0.003572" rpy="0.0 0.0 0.0"/>
-          <inertia ixx="0.058902" ixy="0.000000" ixz="0.000001"
-                                  iyy="0.056884" iyz="-0.003672"
-                                                 izz="0.034271"/>
-      </inertial>
     </link>
     <link name="${prefix}link_4">
@@ -106,11 +78,4 @@
         </geometry>
       </collision>
-      <inertial>
-          <mass value="4.54015"/>
-          <origin xyz="-0.002488 0.049988 0.296156" rpy="0.0 0.0 0.0"/>
-          <inertia ixx="0.043246" ixy="0.000003" ixz="-0.000683"
-                                  iyy="0.038394" iyz="-0.000004"
-                                                 izz="0.014525"/>
-      </inertial>
     </link>
     <link name="${prefix}link_5">
@@ -128,11 +93,4 @@
         </geometry>
       </collision>
-      <inertial>
-          <mass value="0.56876"/>
-          <origin xyz="0.000000 0.049931 0.222823" rpy="0.0 0.0 0.0"/>
-          <inertia ixx="0.001084" ixy="0.000000" ixz="0.000000"
-                                  iyy="0.001123" iyz="0.000001"
-                                                 izz="0.000383"/>
-      </inertial>
     </link>
     <link name="${prefix}link_6">
@@ -150,13 +108,6 @@
         </geometry>
       </collision>
-      <inertial>
-          <mass value="0.03098"/>
-          <origin xyz="-0.000243 0.050000 -0.006293" rpy="0.0 0.0 0.0"/>
-          <inertia ixx="0.000012" ixy="0.000000" ixz="0.000000"
-                                  iyy="0.000011" iyz="0.000000"
-                                                 izz="0.000022"/>
-      </inertial>
     </link>
-    <!-- joints: main serial chain -->
+    <link name="${prefix}tool0" />
     <joint name="${prefix}joint_1" type="revolute">
       <origin xyz="0 0 0.330" rpy="0 0 0" />
@@ -165,7 +116,6 @@
       <axis xyz="0 0 1" />
       <limit effort="0" lower="-2.965" upper="2.965" velocity="7.85" />
-      <dynamics damping="0.0" friction="0.0"/>
-   </joint>
-   <joint name="${prefix}joint_2" type="revolute">
+    </joint>
+    <joint name="${prefix}joint_2" type="revolute">
       <origin xyz="0.050 0 0" rpy="0 0 0"/>
       <parent link="${prefix}link_1" />
@@ -199,8 +149,13 @@
       <parent link="${prefix}link_5"/>
       <child link="${prefix}link_6"/>
-      <axis xyz="-1 0 0"/>
+      <axis xyz="1 0 0"/>
       <limit effort="0" lower="-6.285" upper="6.285" velocity="17.45" />
     </joint>
-    <!-- ROS-Industrial 'base' frame: base_link to Fanuc World Coordinates transform -->
+    <joint name="${prefix}joint_6-tool0" type="fixed">
+      <origin xyz="0 0 0" rpy="${m_pi} ${-m_pi_2} 0" />
+      <parent link="${prefix}link_6" />
+      <child link="${prefix}tool0" />
+    </joint>
+    <!-- ROS base_link to Fanuc World Coordinates transform -->
     <link name="${prefix}base" />
     <joint name="${prefix}base_link-base" type="fixed">
@@ -209,18 +164,4 @@
       <child link="${prefix}base"/>
     </joint>
-    <!-- ROS-Industrial 'flange' frame: attachment point for EEF models -->
-    <link name="${prefix}flange" />
-    <joint name="${prefix}joint_6-flange" type="fixed">
-      <origin xyz="0 0 0" rpy="0 0 0" />
-      <parent link="${prefix}link_6" />
-      <child link="${prefix}flange" />
-    </joint>
-    <!-- ROS-Industrial 'tool0' frame: all-zeros tool frame -->
-    <link name="${prefix}tool0" />
-    <joint name="${prefix}link_6-tool0" type="fixed">
-      <origin xyz="0 0 0" rpy="${pi} ${-pi/2.0} 0" />
-      <parent link="${prefix}flange" />
-      <child link="${prefix}tool0" />
-    </joint>
   </xacro:macro>
 </robot>
